Commit message: Add files via upload

File: open_manipulator_description/urdf/open_manipulator.urdfscoop.xacro (robot description, xacro)
@@ -150,9 +150,9 @@
   </link>
   <!--  Gripper joint -->
-  <joint name="gripper" type="revolute">
+  <joint name="gripper" type="prismatic">
     <parent link="link5"/>
     <child link="gripper_link"/>
-    <origin xyz="0.1 0 0.015" rpy="0 1.571 0"/>
-    <axis xyz="1 0 0"/>
+    <origin xyz="0.0750 0 0.03" rpy="1.57078 3.14 -1.57078"/>
+    <axis xyz="0 1 0"/>
     <limit velocity="4.8" effort="1" lower="-0.010" upper="0.019" />
   </joint>
