Commit message: Add files via upload
Mesh files and URDF files updated for shovel end effector

File: open_manipulator_description/urdf/open_manipulator.urdf.xacro (robot description, xacro)
@@ -153,5 +153,5 @@
     <parent link="link5"/>
     <child link="gripper_link"/>
-    <origin xyz="0.0817 0.021 0.0" rpy="0 0 0"/>
+    <origin xyz="0.0750 0 0.03" rpy="1.57078 3.14 -1.57078"/>
     <axis xyz="0 1 0"/>
     <limit velocity="4.8" effort="1" lower="-0.010" upper="0.019" />

Commit message: Add files via upload
open_manipulator.urdf.xacro is the correct joint and position for the barrel, open_manipulator.urdfscoop.xacro is the correct joint and position of the scoop

File: open_manipulator_description/urdf/open_manipulator.urdf.xacro (robot description, xacro)
@@ -150,10 +150,10 @@
   </link>
   <!--  Gripper joint -->
-  <joint name="gripper" type="revolute">
+  <joint name="gripper" type="continuous">
     <parent link="link5"/>
     <child link="gripper_link"/>
     <origin xyz="0.1 0 0.015" rpy="0 1.571 0"/>
     <axis xyz="1 0 0"/>
-    <limit velocity="4.8" effort="1" lower="-0.010" upper="0.019" />
+    <limit velocity="50" effort="1" lower="${-pi*0.57}" upper="${pi*0.65}" />
   </joint>
   <!--  Gripper link -->
@@ -181,9 +181,9 @@
   </link>
   <!--  Gripper joint sub -->
-  <joint name="gripper_sub" type="prismatic">
+  <joint name="gripper_sub" type="revolute">
     <parent link="link5"/>
     <child link="gripper_link_sub"/>
     <origin xyz="0.0817 -0.021 0" rpy="0 0 0"/>
-    <axis xyz="0 -1 0"/>
+    <axis xyz="0 1 0"/>
     <limit velocity="4.8" effort="1" lower="-0.010" upper="0.019" />
     <mimic joint="gripper" multiplier="1"/>

File: open_manipulator_description/urdf/open_manipulator.urdfscoop.xacro (robot description, xacro)
@@ -150,8 +150,8 @@
   </link>
   <!--  Gripper joint -->
-  <joint name="gripper" type="prismatic">
+  <joint name="gripper" type="resolute">
     <parent link="link5"/>
     <child link="gripper_link"/>
-    <origin xyz="0.0750 0 0.03" rpy="1.57078 3.14 -1.57078"/>
+    <origin xyz="0.075 0 0.03" rpy="1.57078 1.57078 -1.57078"/>
     <axis xyz="0 1 0"/>
     <limit velocity="4.8" effort="1" lower="-0.010" upper="0.019" />
@@ -160,5 +160,5 @@
   <link name="gripper_link">
     <visual>
-      <origin xyz="0.0 0.0 0" rpy="0 0 0"/>
+      <origin xyz="0 0 0" rpy="0 0 0"/>
       <geometry>
         <mesh filename="package://open_manipulator_description/meshes/chain_link_grip_l.stl" scale="0.001 0.001 0.001"/>
@@ -181,9 +181,9 @@
   </link>
   <!--  Gripper joint sub -->
-  <joint name="gripper_sub" type="prismatic">
+  <joint name="gripper_sub" type="revolute">
     <parent link="link5"/>
     <child link="gripper_link_sub"/>
-    <origin xyz="0.0817 -0.021 0" rpy="0 0 0"/>
-    <axis xyz="0 -1 0"/>
+    <origin xyz="0 0 0" rpy="0 0 0"/>
+    <axis xyz="0 1 0"/>
     <limit velocity="4.8" effort="1" lower="-0.010" upper="0.019" />
     <mimic joint="gripper" multiplier="1"/>
@@ -192,5 +192,5 @@
   <link name="gripper_link_sub">
     <visual>
-      <origin xyz="0.0 -0.0 0" rpy="0 0 0"/>
+      <origin xyz="0 0.0 0" rpy="0 0 0"/>
       <geometry>
         <mesh filename="package://open_manipulator_description/meshes/chain_link_grip_r.stl" scale="0.001 0.001 0.001"/>
@@ -214,5 +214,5 @@
   <!-- end effector joint -->
   <joint name="end_effector_joint" type="fixed">
-    <origin xyz="0.126 0.0 0.0" rpy="0 0 0"/>
+    <origin xyz="1 0.0 0.0" rpy="0 0 0"/>
     <parent link="link5"/>
     <child link="end_effector_link"/>
